File: Adafruit-Feather.brd (EAGLE design)
At the start: 50.8 x 22.9 mm, 39 parts, among them IC1 CP2104, Q1 mmbt2222, Q2 mmbt2222, Q3 DMG3415U, SW2 KMR2, U2 AP2112-3.3, U3 MCP73831T-2ACI/OT, X1 JSTPH, X4 20329

Commit message: modified files again
Connections:
- removed net RXD0: IC1.21
- removed net TXD0: IC1.20
- new net REGIN: IC1.7
- new net VDD: IC1.6
- new net VIO: IC1.5
- net 3.3V: no longer IC1.5, IC1.6, IC1.7
- net DTR: no longer IC1.23
- net N$2: no longer IC1.3
- net N$6: no longer IC1.4
- net RTS: no longer IC1.19
Routing:
- net RXD0: track 33.4 -> 0.00 mm, vias 2 -> 0
- net TXD0: track 26.7 -> 0.00 mm, vias 2 -> 0
- net 3.3V: track 80.1 -> 76.2 mm
- net GND: track 27.6 -> 24.7 mm, vias 56 -> 55
- net VBUS: track 56.2 -> 55.3 mm
- net DTR: track 13.9 -> 13.1 mm
- net N$6: track 5.16 -> 4.43 mm
- net N$2: track 5.33 -> 4.77 mm
